File: hardware/power-module.kicad_sch (KiCad schematic)
At the start: 36 parts, among them CN1 WJ2EDGRC-5.08-2P, K1 SRA-9VDC-CL, K2 SRA-9VDC-CL, K5 SRA-9VDC-CL, K6 SRA-9VDC-CL, Q1 SS8050_C2150, Q2 SS8050_C2150, U1 MIC5205-3.3YM5-MS, U2 PM254-2-05-W-8.5, U3 CC6903SO-10A, U4 ESP32-C3-MINI-1, U5 XC6206P332MR_C5148692, U6 L7809CV_C347291

Commit message: Add PoE board
Parts:
- removed C3: 1uF, Capacitor_SMD:C_0603_1608Metric, symbol Device:C
- removed D1: MB10FH5G0NP, LCSC:MBF_L4.8-W3.9-P2.50-LS6.7-TR, symbol LCSC:MB10FH5G0NP
- removed H1: 2*5P header, LCSC:HDR-TH_10P-P2.54-H-M-R2-C5-S2.54-W12.9, symbol easyeda2kicad:2*5Pheader
- removed K1, K2, K5, K6: SRA-9VDC-CL, LCSC:RELAY-TH_SRA-9VDC-CL, symbol LCSC:SRA-9VDC-CL
- removed LED4: XL-1608UYC-06, LCSC:LED0603-RD-YELLOW, symbol easyeda2kicad:XL-1608UYC-06
- removed R9: 120, Resistor_SMD:R_0603_1608Metric, symbol Device:R
- removed U2: PM254-2-05-W-8.5, LCSC:HDR-TH_10P-P2.54-H-F-R2-C5-W8.5, symbol easyeda2kicad:PM254-2-05-W-8.5
- removed U3: CC6903SO-10A, LCSC:SOP-8_L4.9-W3.9-P1.27-LS6.0-BL, symbol easyeda2kicad:CC6903SO-10A
- removed U4: ESP32-C3-MINI-1, PCM_Espressif:ESP32-C3-MINI-1, symbol PCM_Espressif:ESP32-C3-MINI-1
- removed U6: L7809CV_C347291, LCSC:TO-220-3_L10.0-W4.5-P2.54-L, symbol LCSC:L7809CV_C347291
- added C10, C11, C12, C13, C14, C15: 0.1uF, Capacitor_SMD:C_0603_1608Metric, symbol Device:C
- added C3: 100uF 25V, Capacitor_SMD:C_0603_1608Metric, symbol Device:C
- added C3: 1uF, Capacitor_SMD:C_0603_1608Metric, symbol Device:C
- added C6, C7, C8: 4.7uF, Capacitor_SMD:C_0603_1608Metric, symbol Device:C
- added K1, K2, K3, K4: SRA-12VDC-CL, easyeda2kicad:RELAY-TH_SRA-X-CX, symbol easyeda2kicad:SRA-12VDC-CL
- added P1: WJ2EDGRC-5.08-4P, easyeda2kicad:CONN-TH_4P-P5.08_WJ2EDGRC-5.08-4P, symbol easyeda2kicad:WJ2EDGRC-5.08-4P
- added R2 (x3): 10K, Resistor_SMD:R_0603_1608Metric, symbol Device:R
- added R2: 56, Resistor_SMD:R_0603_1608Metric, symbol Device:R
- added RJ1: HY931147C, easyeda2kicad:RJ45-TH_HY931147C, symbol easyeda2kicad:HY931147C
- added U10, U11, U12, U6, U8, U9: XL-1010RGBC-WS2812B, easyeda2kicad:LED-SMD_4P-L1.0-W1.0-TL_XL-1010RGBC-WS2812B, symbol easyeda2kicad:XL-1010RGBC-WS2812B
- added U2: CC6903SO-10A, easyeda2kicad:SOP-8_L4.9-W3.9-P1.27-LS6.0-BL, symbol easyeda2kicad:CC6903SO-10A
- added U3: W5500, easyeda2kicad:LQFP-48_L7.0-W7.0-P0.50-LS9.0-BL, symbol easyeda2kicad:W5500
- added U4: ESP32-C3FH4, easyeda2kicad:QFN-32_L5.0-W5.0-P0.50-TL-EP3.7, symbol easyeda2kicad:ESP32-C3FH4
- added U7: DP9900LP-12V, easyeda2kicad:PWRM-TH_DP9900LP-5V, symbol easyeda2kicad:DP9900LP-12V
- added X1: X49SM25MSD2SC, easyeda2kicad:HC-49S_L11.4-W4.8, symbol easyeda2kicad:X49SM25MSD2SC
- C4: value 330nF -> 10uF 25V
- C5: value 100nF -> 4.7uF
- CN1: footprint LCSC:CONN-TH_2P-P5.08_WJ2EDGRC-5.08-2P -> easyeda2kicad:CONN-TH_2P-P5.08_WJ2EDGRC-5.08-2P
- R4: value 10k -> 56
- R5: value 10k -> 12.4K 1%
- R6: value 10k -> 1M
- U1: footprint LCSC:SOT-23-5_L2.9-W1.6-P0.95-LS2.8-BR -> easyeda2kicad:SOT-23-5_L2.9-W1.6-P0.95-LS2.8-BR
Connections:
- net BOOT: now also U4.14 (GPIO8)
- net CONTROLLER POWER IN: no longer C2.1, R3.1, R4.1, R5.2, R6.2, U1.5 (OUT)
- net CURRENT SENSING INPUT: now also U2.7 (OUT)
- net GND: now also C4.1, R5.2, C10.2, C11.2, C12.2, C13.2, C14.2, C15.2, C3.1, C3.1, C6.2, C7.2, C8.2, R2.1, RJ1.12, RJ1.14, RJ1.GND1 (GND), RJ1.GND2 (GND), U10.3 (GND), U11.3 (GND), U12.3 (GND), U2.5 (GND), U3.14 (AGND), U3.16 (AGND), U3.19 (AGND), U3.23 (RSVD), U3.29 (GND), U3.3 (AGND), U3.48 (AGND), U3.9 (AGND), U4.33 (EP), U6.3 (GND), U7.3 (-VDC), U8.3 (GND), U9.3 (GND); no longer C4.2
- net RELAY POWER: now also K1.4, K2.3, K3.4, K4.3; no longer C5.1
- net RESET: now also C3.2, R2.1, U4.7 (CHIP_EN); no longer R4.2
- net TRACK OUT A: now also K3.5, P1.2, P1.4
- net TRACK OUT B: now also K4.5, P1.1, P1.3; no longer CN1.1
- net TRACK POWER A: now also CN1.2, K1.5
- net TRACK POWER B: now also K2.5, U2.1 (IP+), U2.2 (IP+)
- net TRACK POWER ENABLED A: now also K1.1, K3.2, K4.1
- net TRACK POWER ENABLED B: now also K2.1, K3.1, K4.2
- net USB +: now also U4.26 (GPIO19)
- net USB -: now also U4.25 (GPIO18)
- net at R6.1: now also C8.1, U3.31 (XO), X1.1 (OSC1)
- net at R5.1: now also U3.10 (EXRES1)
- net at D2.2 (A), Q2.3 (C): now also K1.3, K2.4
- net at D3.2 (A), Q1.3 (C): now also K3.3, K4.4
- net TRACK POWER IN renamed +12V
- net +12V: now also C4.2, C3.2, U7.1 (+VDC), U7.2 (+VDC); no longer C4.1
- new net: C7.1, R6.2, U3.30 (XI/CLKIN), X1.2 (OSC2)
- new net: R4.1, RJ1.13
- new net: U11.1 (DOUT), U12.4 (DIN)
- new net: U10.1 (DOUT), U11.4 (DIN)
- new net: C6.1, U3.22 (1V2O)
- new net: U6.1 (DOUT), U8.4 (DIN)
- new net: R2.2, U4.15 (GPIO9)
- new net: R2.1, RJ1.11
- new net: C5.1, U3.20 (TOCAP)
- new net: CN1.1, U2.3 (IP-), U2.4 (IP-)
- new net: U10.4 (DIN), U9.1 (DOUT)
- new net: U8.1 (DOUT), U9.4 (DIN)
- new net +3.3V: C2.1, R2.2, R2.2, R3.1, U1.5 (OUT), U2.8 (VCC), U3.11 (AVDD), U3.15 (AVDD), U3.17 (AVDD), U3.21 (AVDD), U3.28 (VDD), U3.4 (AVDD), U3.8 (AVDD), U4.11 (VDD3P3_RTC), U4.17 (VDD3P3_CPU), U4.18 (VDD_SPI), U4.2 (VDD3P3), U4.3 (VDD3P3), U4.31 (VDDA), U4.32 (VDDA)
- new net +5V: C10.1, C11.1, C12.1, C13.1, C14.1, C15.1, U10.2 (VDD), U11.2 (VDD), U12.2 (VDD), U6.2 (VDD), U8.2 (VDD), U9.2 (VDD)
- new net ETHERNET RX +: RJ1.2, U3.6 (RXP)
- new net ETHERNET RX -: RJ1.1, U3.5 (RXN)
- new net ETHERNET TX +: RJ1.6, U3.2 (TXP)
- new net ETHERNET TX -: RJ1.5, U3.1 (TXN)
- new net LED ACTIVITY: R2.2, U3.27 (ACTLED)
- new net LED DATA IN: U6.4 (DIN)
- new net LED LINK: R4.2, U3.25 (LINKLED)
- new net POE IN +: RJ1.9, U7.5 (VIN+), U7.6 (VIN+)
- new net POE IN -: RJ1.10, U7.7 (VIN-), U7.8 (VIN-)
- new net WIZ INTERRUPT: U3.36 (INTn)
- new net WIZ RESET: U3.37 (RSTn)
- new net WIZ SPI CS: U3.32 (SCSn), U4.16 (GPIO10)
- new net WIZ SPI MISO: R2.1, U3.34 (MISO), U4.6 (GPIO2)
- new net WIZ SPI MOSI: U3.35 (MOSI), U4.13 (MTDO)
- new net WIZ SPI SCLK: U3.33 (SCLK), U4.12 (MTCK)
- no-connect marks 8 -> 35
Other:
- note added: "Sensor supports current in both directions"
- moved on the sheet: C1, C2, D2, D3, H2, LED1, LED2, LED5, Q1, Q2, R1, R10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

Commit message: Add routes and part placement
Parts:
- removed D3: BAS321,115, LCSC:SOD-323_L1.8-W1.3-LS2.5-RD, symbol easyeda2kicad:BAS321,115
- removed H2: DZ127R-11-06-25, LCSC:HDR-TH_6P-P1.27-V-M-A, symbol easyeda2kicad:DZ127R-11-06-25
- removed LED5: XL-1608UYC-06, LCSC:LED0603-RD-YELLOW, symbol easyeda2kicad:XL-1608UYC-06
- removed Q1, Q2: SS8050_C2150, LCSC:SOT-23-3_L2.9-W1.3-P1.90-LS2.4-BR, symbol LCSC:SS8050_C2150
- added C18: 0.33uF, Capacitor_SMD:C_0603_1608Metric, symbol Device:C
- added C19, C28, C29, C3 (x3), C30, C31: 0.1uF, Capacitor_SMD:C_0603_1608Metric, symbol Device:C
- added C20: 0.1nF, Capacitor_SMD:C_0603_1608Metric, symbol Device:C
- added C3: 10uF, Capacitor_SMD:C_0603_1608Metric, symbol Device:C
- added C3: 10nF, Capacitor_SMD:C_0603_1608Metric, symbol Device:C
- added C3 (x4): 1uF, Capacitor_SMD:C_0603_1608Metric, symbol Device:C
- added D1: BAS321,115, easyeda2kicad:SOD-323_L1.8-W1.3-LS2.5-RD, symbol easyeda2kicad:BAS321,115
- added H1: DZ127R-11-06-25, easyeda2kicad:HDR-TH_6P-P1.27-V-M-A, symbol easyeda2kicad:DZ127R-11-06-25
- added J1: Conn_01x04_Pin, Connector_PinHeader_2.54mm:PinHeader_1x04_P2.54mm_Vertical, symbol Connector:Conn_01x04_Pin
- added L1: 2.0nH, Inductor_SMD:L_0603_1608Metric, symbol Device:L
- added LED3: XL-1608UYC-06, easyeda2kicad:LED0603-RD-YELLOW, symbol easyeda2kicad:XL-1608UYC-06
- added Q1, Q2: SS8050_C2150, easyeda2kicad:SOT-23-3_L2.9-W1.3-P1.90-LS2.4-BR, symbol easyeda2kicad:SS8050_C2150
- added U13: L327S400H11L, easyeda2kicad:CRYSTAL-SMD_4P-L3.2-W2.5-BL, symbol easyeda2kicad:L327S400H11L
- added U14: UMW78L05, easyeda2kicad:SOT-89-3_L4.5-W2.5-P1.50-LS4.2-BR, symbol easyeda2kicad:UMW78L05
- added U15, U16, U17, U18: XL-1010RGBC-WS2812B, easyeda2kicad:LED-SMD_4P-L1.0-W1.0-TL_XL-1010RGBC-WS2812B, symbol easyeda2kicad:XL-1010RGBC-WS2812B
- D2: footprint LCSC:SOD-323_L1.8-W1.3-LS2.5-RD -> easyeda2kicad:SOD-323_L1.8-W1.3-LS2.5-RD
- LED1, LED2: footprint LCSC:LED0603-RD-YELLOW -> easyeda2kicad:LED0603-RD-YELLOW
- U5: footprint LCSC:SOT-23-3_L2.9-W1.3-P1.90-LS2.4-BR -> easyeda2kicad:SOT-23-3_L2.9-W1.3-P1.90-LS2.4-BR
Connections:
- net CONTROLLER POWER IN is gone; now on net +3.3V: U5.2 (VOUT)
- net RELAY POWER is gone; now on net +12V: D2.1 (K), K1.4, K2.3, K3.4, K4.3
- net +12V: now also C18.1, D1.1 (K), J1.2 (Pin_2), U14.3 (IN)
- net +3.3V: now also C20.1, C3.1, C3.2, C3.2, C3.2, J1.3 (Pin_3); no longer U4.18 (VDD_SPI), U4.2 (VDD3P3), U4.3 (VDD3P3)
- net +5V: now also C19.1, C28.1, C29.1, C30.1, C31.1, J1.1 (Pin_1), U14.1 (OUT), U15.2 (VDD), U16.2 (VDD), U17.2 (VDD), U18.2 (VDD)
- net BOOT: now also H1.4
- net CURRENT SENSING INPUT: now also U4.4 (XTAL_32K_P)
- net GND: now also C18.2, C19.2, C20.2, C28.2, C29.2, C3.1, C3.1, C3.1, C3.1, C3.1, C3.1, C3.1, C3.1, C3.2, C30.2, C31.2, H1.6, J1.4 (Pin_4), LED3.1 (K), Q1.2 (E), Q2.2 (E), U13.2 (GND), U13.4 (GND), U14.2 (GND), U15.3 (GND), U16.3 (GND), U17.3 (GND), U18.3 (GND)
- net LED DATA IN: now also R2.2, U4.15 (GPIO9)
- net RESET: now also H1.5
- net TRACK DIRECTION: now also U4.27 (U0RXD)
- net TRACK POWER ENABLE: now also U4.28 (U0TXD)
- net USB +: now also H1.2
- net USB -: now also H1.3
- net WIZ RESET: now also U4.8 (GPIO3)
- net at U5.3 (VIN): now also H1.1
- net at U4.29 (XTAL_N): now also C3.2, U13.3
- net at U4.30 (XTAL_P): now also C3.2, U13.1
- net at R10.1: now also LED3.2 (A)
- net at R1.1: now also Q2.1 (B)
- net at K1.3, K2.4: now also D1.2 (A), Q2.3 (C); no longer D2.2 (A)
- net at K3.3, K4.4: now also D2.2 (A), Q1.3 (C)
- net at R11.1: now also Q1.1 (B)
- net at U12.1 (DOUT): now also U15.4 (DIN)
- net WIZ INTERRUPT: no longer names the net of U3.36 (INTn)
- new net: C3.2, C3.2, L1.2
- new net: C3.2, L1.1, U4.2 (VDD3P3), U4.3 (VDD3P3)
- new net: U17.1 (DOUT), U18.4 (DIN)
- new net: U16.1 (DOUT), U17.4 (DIN)
- new net: U15.1 (DOUT), U16.4 (DIN)
- no-connect marks 35 -> 38
Other:
- note added: "No caps, debug only"
- note added: "Voltage Probe"
- moved on the sheet: C1, C10, C11, C12, C13, C14, C15, C2, C3, C4, C5, C6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

Commit message: Fix SPI pins, power supply current
Parts:
- removed U1: MIC5205-3.3YM5-MS, easyeda2kicad:SOT-23-5_L2.9-W1.6-P0.95-LS2.8-BR, symbol easyeda2kicad:MIC5205-3.3YM5-MS
- removed U5: XC6206P332MR_C5148692, easyeda2kicad:SOT-23-3_L2.9-W1.3-P1.90-LS2.4-BR, symbol easyeda2kicad:XC6206P332MR_C5148692
- added U1, U5: AMS1117-3.3_C347222, easyeda2kicad:SOT-223-4_L6.5-W3.5-P2.30-LS7.0-BR, symbol easyeda2kicad:AMS1117-3.3_C347222
- C1: value 1uF -> 0.1nF
- C2: value 2.2uF -> 0.1nF
Connections:
- net +12V: now also C2.1, U1.3 (VIN); no longer C1.1
- net +3.3V: now also C1.1, U1.2 (VOUT(TAB)), U5.2 (VOUT(TAB)); no longer C2.1
- net BOOT: now also U4.15 (GPIO9); no longer U4.14 (GPIO8)
- net GND: now also U1.1 (ADJ(GND)), U5.1 (ADJ(GND))
- net LED DATA IN: now also U4.16 (GPIO10); no longer R2.2, U4.15 (GPIO9)
- net WIZ SPI CS: now also U4.13 (MTDO); no longer U4.16 (GPIO10)
- net WIZ SPI MISO: now also U4.10 (MTDI); no longer R2.1, U4.6 (GPIO2)
- net WIZ SPI MOSI: now also U4.12 (MTCK); no longer U4.13 (MTDO)
- net WIZ SPI SCLK: now also U4.9 (MTMS); no longer U4.12 (MTCK)
- net at H1.1: now also U5.3 (VIN)
- new net: R2.1, U4.6 (GPIO2)
- new net: R2.2, U4.14 (GPIO8)
- no-connect marks 38 -> 37
Other:
- moved on the sheet: C3, L1, LED1, R2, R3, U13, U4

Commit message: Fix crystal
Parts:
- removed X1: X49SM25MSD2SC, easyeda2kicad:HC-49S_L11.4-W4.8, symbol easyeda2kicad:X49SM25MSD2SC
- added C3: 1uF, Capacitor_SMD:C_0603_1608Metric, symbol Device:C
- added C32: TAJE337M016RNJ, easyeda2kicad:CAP-SMD_L7.3-W4.3-R-RD, symbol easyeda2kicad:TAJE337M016RNJ
- added J2, J3, J4: Conn_01x02, Connector_PinHeader_2.54mm:PinHeader_1x02_P2.54mm_Vertical, symbol Connector_Generic:Conn_01x02
- added L2: 24nH, Inductor_SMD:L_0603_1608Metric, symbol Device:L
- added R13: 6.2k, Resistor_SMD:R_0603_1608Metric, symbol Device:R
- added X1: X322525MRB4SI, easyeda2kicad:OSC-SMD_4P-L3.2-W2.5-BL_SIT8008BI, symbol easyeda2kicad:X322525MRB4SI
- C3: value 1uF -> 14pF
- C7, C8: value 4.7uF -> 18pF
Connections:
- net +12V: now also J4.2 (Pin_2)
- net +3.3V: now also U4.18 (VDD_SPI), C3.1
- net GND: now also C3.2, C32.2, R13.2, X1.2 (GND), X1.4 (GND)
- net POE IN +: now also J3.2 (Pin_2); no longer RJ1.9
- net POE IN -: now also J2.1 (Pin_1); no longer RJ1.10
- net at C3.2, U13.1: now also L2.2; no longer U4.30 (XTAL_P)
- net at C7.1, R6.2, U3.30 (XI/CLKIN): now also X1.1 (OSC1)
- net at C8.1, R6.1, U3.31 (XO): now also X1.3 (OSC2)
- new net: C32.1, J4.1 (Pin_1), R13.1
- new net: L2.1, U4.30 (XTAL_P)
- new net: J2.2 (Pin_2), RJ1.10
- new net: J3.1 (Pin_1), RJ1.9
- no-connect marks 37 -> 36
Other:
- moved on the sheet: C3, C7, C8, R2, R4, R6, RJ1, U13

Commit message: Add current sensing input capactior
Parts:
- added C3: 0.1uF, Capacitor_SMD:C_0603_1608Metric, symbol Device:C
Connections:
- net CURRENT SENSING INPUT: now also C3.2
- net GND: now also C3.1
Changed lines of the file:
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@@
   (junction (at 289.56 257.81) (diameter 0) (color 0 0 0 0)
   )
+  (junction (at 412.75 38.1) (diameter 0) (color 0 0 0 0)
+  )
   (junction (at 330.2 252.73) (diameter 0) (color 0 0 0 0)
   )
@@
     (stroke (width 0) (type default))
   )
+  (wire (pts (xy 401.32 38.1) (xy 402.59 38.1))
+    (stroke (width 0) (type default))
+  )
   (wire (pts (xy 400.05 207.01) (xy 400.05 198.12))
     (stroke (width 0) (type default))
@@
     (stroke (width 0) (type default))
   )
-  (wire (pts (xy 414.02 63.5) (xy 414.02 78.74))
+  (wire (pts (xy 412.75 25.4) (xy 412.75 38.1))
     (stroke (width 0) (type default))
   )
@@
     (stroke (width 0) (type default))
   )
+  (wire (pts (xy 410.21 38.1) (xy 412.75 38.1))
+    (stroke (width 0) (type default))
+  )
   (wire (pts (xy 525.78 123.19) (xy 515.62 123.19))
     (stroke (width 0) (type default))
@@
     (stroke (width 0) (type default))
   )
+  (wire (pts (xy 412.75 38.1) (xy 412.75 78.74))
+    (stroke (width 0) (type default))
+  )
   (wire (pts (xy 332.74 349.25) (xy 349.25 349.25))
     (stroke (width 0) (type default))
@@
     (stroke (width 0) (type default))
   )
-  (wire (pts (xy 414.02 78.74) (xy 425.45 78.74))
+  (wire (pts (xy 412.75 78.74) (xy 425.45 78.74))
     (stroke (width 0) (type default))
   )
@@
     (effects (font (size 1.27 1.27)) (justify left bottom))
   )
-  (label "CURRENT SENSING INPUT" (at 414.02 63.5 90) (fields_autoplaced)
+  (label "CURRENT SENSING INPUT" (at 412.75 25.4 0) (fields_autoplaced)
     (effects (font (size 1.27 1.27)) (justify left bottom))
   )
@@
     )
   )
+  (symbol (lib_id "power:GND") (at 401.32 38.1 270) (unit 1)
+    (in_bom yes) (on_board yes) (dnp no) (fields_autoplaced)
+    (property "Reference" "#PWR071" (at 394.97 38.1 0)
+      (effects (font (size 1.27 1.27)) hide)
+    )
+    (property "Value" "GND" (at 397.51 38.1 90)
+      (effects (font (size 1.27 1.27)) (justify right))
+    )
+    (property "Footprint" "" (at 401.32 38.1 0)
+      (effects (font (size 1.27 1.27)) hide)
+    )
+    (property "Datasheet" "" (at 401.32 38.1 0)
+      (effects (font (size 1.27 1.27)) hide)
+    )
+    (pin "1")
+    (instances
+      (project "power-module"
+        (path "/89207206-eadb-4092-9709-787055aa952e"
+          (reference "#PWR071") (unit 1)
+        )
+      )
+    )
+  )
   (symbol (lib_id "easyeda2kicad:XL-1010RGBC-WS2812B") (at 146.05 361.95 0) (unit 1)
     (in_bom yes) (on_board yes) (dnp no)
@@
         )
       )
+    )
+  )
+  (symbol (lib_id "Device:C") (at 406.4 38.1 90) (unit 1)
+    (in_bom yes) (on_board yes) (dnp no) (fields_autoplaced)
+    (property "Reference" "C3" (at 406.4 30.48 90)
+      (effects (font (size 1.27 1.27)))
+    )
+    (property "Value" "0.1uF" (at 406.4 33.02 90)
+      (effects (font (size 1.27 1.27)))
+    )
+    (property "Footprint" "Capacitor_SMD:C_0603_1608Metric" (at 410.21 37.1348 0)
+      (effects (font (size 1.27 1.27)) hide)
+    )
+    (property "Datasheet" "~" (at 406.4 38.1 0)
+      (effects (font (size 1.27 1.27)) hide)
+    )
+    (pin "1")
+    (pin "2")
+    (instances
+      (project "map-station"
+        (path "/1354031f-3471-4ffd-8514-54815221ed33"
+          (reference "C3") (unit 1)
+        )
+      )
+      (project "power-module"
+        (path "/89207206-eadb-4092-9709-787055aa952e"
+          (reference "C34") (unit 1)
+        )
+      )
